Commit message: feat: add some test and update param

File: src/robot_description/urdf/robot_description.urdf (robot description, URDF)
Before this commit: robot robot_description, 6 links, 5 joints
Joints:
- joint left_wheel_jl: origin xyz=-0.000275319332503843 0.0780325399548871 -0.0266929866933577 rpy=0 0 0 -> xyz=-0.000275319332503843 0.105 -0.0266929866933577 rpy=0 0 0
- joint right_wheel_jl: origin xyz=-0.000172826687894733 -0.0780325399548871 -0.0273779601243553 rpy=0 0 0 -> xyz=-0.000172826687894733 -0.105 -0.0273779601243553 rpy=0 0 0

Commit message: fix: update urdf

File: src/robot_description/urdf/robot_description.urdf (robot description, URDF)
Before this commit: robot robot_description, 6 links, 5 joints
Joints:
- joint lidar_jl: origin xyz=0.000149 0.00018885 0.0763 rpy=0 0 0 -> xyz=0.000149 0.00018885 0.0763 rpy=0 0 3.14159

Commit message: fix: robot wheel distance

File: src/robot_description/urdf/robot_description.urdf (robot description, URDF)
Before this commit: robot robot_description, 6 links, 5 joints
Joints:
- joint left_wheel_jl: origin xyz=-0.000275319332503843 0.105 -0.0266929866933577 rpy=0 0 0 -> xyz=-0.000275319332503843 0.102 -0.0266929866933577 rpy=0 0 0
- joint right_wheel_jl: origin xyz=-0.000172826687894733 -0.105 -0.0273779601243553 rpy=0 0 0 -> xyz=-0.000172826687894733 -0.102 -0.0273779601243553 rpy=0 0 0
